File: HARDWARE/MINIHATv.0/Ethernet.kicad_sch (KiCad schematic)
At the start: 32 parts, among them J1 8P8C_LED_Shielded, U1 LAN8742A, Y1 Crystal_GND24_Small

Commit message: buses defined ind project settings, added stm antenna footprint, organized TOP
Changed lines of the file:
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@@
 		)
 	)
-	(hierarchical_label "RMII{TXD0 TXD1 TXDEN RXD0 RXD1 RXER CRS_DV MDIO MDC}"
+	(hierarchical_label "RMII"
 		(shape input)
 		(at 31.75 71.12 180)

Commit message: added i2c for hdmi
Parts:
- renumbered C8 to C12, C1 to C13, C2 to C14, C10 to C15, C4 to C16, C5 to C17, C6 to C18, C7 to C19, C3 to C20, J1 to J3, R9 to R10, R2 to R11, R3 to R12, R4 to R13, R5 to R14, R6 to R15, R7 to R16, R8 to R17, R1 to R18, R11 to R19, R12 to R20, R13 to R21, R14 to R22, R17 to R23, R18 to R24, R19 to R25, R20 to R26, R15 to R27, R16 to R28, U1 to U5
