File: HARDWARE/MINIHATv.0/QSPI.kicad_sch (KiCad schematic)
At the start: 9 parts, among them U7 W25Q128JVS

Commit message: buses defined ind project settings, added stm antenna footprint, organized TOP
Changed lines of the file:
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@@
 		)
 	)
-	(hierarchical_label "QSPI{CS CLK D0 D1 D2 D3}"
+	(hierarchical_label "QSPI"
 		(shape input)
 		(at 96.52 78.74 180)

Commit message: added i2c for hdmi
Parts:
- renumbered C41 to C51, R43 to R69, R44 to R70, R45 to R71, R46 to R72, R47 to R73, R48 to R74, R49 to R75, U7 to U8
Changed lines of the file:
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@@
 		(in_pos_files yes)
 		(dnp no)
-		(property "Reference" "R45"
+		(property "Reference" "R71"
 			(at 122.682 88.9 90)
 			(show_name no)
@@
 			(project "MINIHATv.0"
 				(path "/19041ef4-1d16-4363-8780-721ad9f20b33/d9e9bbbe-4127-4d38-93b1-ae9f05da8ec2"
-					(reference "R45")
+					(reference "R71")
 					(unit 1)
 				)
@@
 		(dnp no)
 		(fields_autoplaced yes)
-		(property "Reference" "#PWR028"
+		(property "Reference" "#PWR0114"
 			(at 156.21 64.77 0)
 			(hide yes)
@@
 			(project "MINIHATv.0"
 				(path "/19041ef4-1d16-4363-8780-721ad9f20b33/d9e9bbbe-4127-4d38-93b1-ae9f05da8ec2"
-					(reference "#PWR028")
+					(reference "#PWR0114")
 					(unit 1)
 				)
@@
 		(dnp no)
 		(fields_autoplaced yes)
-		(property "Reference" "#PWR029"
+		(property "Reference" "#PWR0113"
 			(at 146.05 81.28 0)
 			(hide yes)
@@
 			(project "MINIHATv.0"
 				(path "/19041ef4-1d16-4363-8780-721ad9f20b33/d9e9bbbe-4127-4d38-93b1-ae9f05da8ec2"
-					(reference "#PWR029")
+					(reference "#PWR0113")
 					(unit 1)
 				)
@@
 		(in_pos_files yes)
 		(dnp no)
-		(property "Reference" "R48"
+		(property "Reference" "R74"
 			(at 122.682 96.52 90)
 			(show_name no)
@@
 			(project "MINIHATv.0"
 				(path "/19041ef4-1d16-4363-8780-721ad9f20b33/d9e9bbbe-4127-4d38-93b1-ae9f05da8ec2"
-					(reference "R48")
+					(reference "R74")
 					(unit 1)
 				)
@@
 		(dnp no)
 		(fields_autoplaced yes)
-		(property "Reference" "C41"
+		(property "Reference" "C51"
 			(at 149.86 68.5799 0)
 			(show_name no)
@@
 			(project "MINIHATv.0"
 				(path "/19041ef4-1d16-4363-8780-721ad9f20b33/d9e9bbbe-4127-4d38-93b1-ae9f05da8ec2"
-					(reference "C41")
+					(reference "C51")
 					(unit 1)
 				)
@@
 		(dnp no)
 		(fields_autoplaced yes)
-		(property "Reference" "#PWR027"
+		(property "Reference" "#PWR0115"
 			(at 156.21 115.57 0)
 			(hide yes)
@@
 			(project "MINIHATv.0"
 				(path "/19041ef4-1d16-4363-8780-721ad9f20b33/d9e9bbbe-4127-4d38-93b1-ae9f05da8ec2"
-					(reference "#PWR027")
+					(reference "#PWR0115")
 					(unit 1)
 				)
@@
 		(in_pos_files yes)
 		(dnp no)
-		(property "Reference" "R46"
+		(property "Reference" "R72"
 			(at 122.682 91.44 90)
 			(show_name no)
@@
 			(project "MINIHATv.0"
 				(path "/19041ef4-1d16-4363-8780-721ad9f20b33/d9e9bbbe-4127-4d38-93b1-ae9f05da8ec2"
-					(reference "R46")
+					(reference "R72")
 					(unit 1)
 				)
@@
 		(in_pos_files yes)
 		(dnp no)
-		(property "Reference" "R43"
+		(property "Reference" "R69"
 			(at 122.682 83.82 90)
 			(show_name no)
@@
 			(project "MINIHATv.0"
 				(path "/19041ef4-1d16-4363-8780-721ad9f20b33/d9e9bbbe-4127-4d38-93b1-ae9f05da8ec2"
-					(reference "R43")
+					(reference "R69")
 					(unit 1)
 				)
@@
 		(in_pos_files yes)
 		(dnp no)
-		(property "Reference" "R49"
+		(property "Reference" "R75"
 			(at 141.732 72.39 0)
 			(show_name no)
@@
 			(project "MINIHATv.0"
 				(path "/19041ef4-1d16-4363-8780-721ad9f20b33/d9e9bbbe-4127-4d38-93b1-ae9f05da8ec2"
-					(reference "R49")
+					(reference "R75")
 					(unit 1)
 				)
@@
 		(in_pos_files yes)
 		(dnp no)
-		(property "Reference" "R47"
+		(property "Reference" "R73"
 			(at 122.682 93.98 90)
 			(show_name no)
@@
 			(project "MINIHATv.0"
 				(path "/19041ef4-1d16-4363-8780-721ad9f20b33/d9e9bbbe-4127-4d38-93b1-ae9f05da8ec2"
-					(reference "R47")
+					(reference "R73")
 					(unit 1)
 				)
@@
 		(dnp no)
 		(fields_autoplaced yes)
-		(property "Reference" "U7"
+		(property "Reference" "U8"
 			(at 167.64 91.4399 0)
 			(show_name no)
@@
 			(project "MINIHATv.0"
 				(path "/19041ef4-1d16-4363-8780-721ad9f20b33/d9e9bbbe-4127-4d38-93b1-ae9f05da8ec2"
-					(reference "U7")
+					(reference "U8")
 					(unit 1)
 				)
@@
 		(in_pos_files yes)
 		(dnp no)
-		(property "Reference" "R44"
+		(property "Reference" "R70"
 			(at 122.682 86.36 90)
 			(show_name no)
@@
 			(project "MINIHATv.0"
 				(path "/19041ef4-1d16-4363-8780-721ad9f20b33/d9e9bbbe-4127-4d38-93b1-ae9f05da8ec2"
-					(reference "R44")
-					(unit 1)
-				)
+					(reference "R70")
+					(unit 1)
+				)
