File: HARDWARE/MINIHATv.0/sdcarad.kicad_sch (KiCad schematic)
At the start: 14 parts, among them J6 Micro_SD_Card_Det2

Commit message: editorial changes
Connections:
- net VDD: now also J6.10 (DET_A)
- net DETECT: no longer names the net of R68.2
- net DETECT: no longer J6.10 (DET_A)

Commit message: repairs on sdcard page connections
Connections:
- net SDIO.DAT0: now also R51.2
- net SDIO.DAT1: now also R54.2
- net SDIO.DAT2: now also R43.2
- net VDD: now also R43.1, R45.1, R48.1, R49.1, R51.1, R54.1, R68.1; no longer J6.10 (DET_A)
- new net DETECT: J6.10 (DET_A)
Changed lines of the file:
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@@
+	)
+	(junction
+		(at 137.16 82.55)
+		(diameter 0)
+		(color 0 0 0 0)
+	)
+	(junction
+		(at 154.94 48.26)
+		(diameter 0)
+		(color 0 0 0 0)
+	)
+	(junction
+		(at 127 55.88)
+		(diameter 0)
+		(color 0 0 0 0)
 	)
 	(junction
@@
 	)
 	(junction
+		(at 137.16 55.88)
+		(diameter 0)
+		(color 0 0 0 0)
+	)
+	(junction
 		(at 106.68 69.85)
 		(diameter 0)
@@
 	)
 	(junction
-		(at 133.35 82.55)
-		(diameter 0)
-		(color 0 0 0 0)
-	)
-	(junction
 		(at 97.79 67.31)
 		(diameter 0)
@@
 	)
 	(junction
-		(at 154.94 48.26)
+		(at 88.9 64.77)
 		(diameter 0)
 		(color 0 0 0 0)
@@
 		(color 0 0 0 0)
 	)
+	(junction
+		(at 127 80.01)
+		(diameter 0)
+		(color 0 0 0 0)
+	)
 	(bus_entry
 		(at 58.42 24.13)
@@
 	)
 	(bus_entry
+		(at 58.42 39.37)
+		(size 2.54 2.54)
+		(stroke
+			(width 0)
+			(type default)
+		)
+	)
+	(bus_entry
 		(at 58.42 36.83)
 		(size 2.54 2.54)
@@
 	(wire
 		(pts
+			(xy 88.9 63.5) (xy 88.9 64.77)
+		)
+		(stroke
+			(width 0)
+			(type default)
+		)
+	)
+	(wire
+		(pts
+			(xy 88.9 64.77) (xy 140.97 64.77)
+		)
+		(stroke
+			(width 0)
+			(type default)
+		)
+	)
+	(wire
+		(pts
 			(xy 60.96 39.37) (xy 73.66 39.37)
 		)
@@
 	(wire
 		(pts
+			(xy 137.16 63.5) (xy 137.16 82.55)
+		)
+		(stroke
+			(width 0)
+			(type default)
+		)
+	)
+	(wire
+		(pts
 			(xy 77.47 69.85) (xy 106.68 69.85)
 		)
@@
 	(wire
 		(pts
+			(xy 60.96 41.91) (xy 73.66 41.91)
+		)
+		(stroke
+			(width 0)
+			(type default)
+		)
+	)
+	(wire
+		(pts
 			(xy 161.29 77.47) (xy 154.94 77.47)
 		)
@@
 	(wire
 		(pts
-			(xy 77.47 80.01) (xy 140.97 80.01)
+			(xy 77.47 80.01) (xy 127 80.01)
 		)
 		(stroke
@@
 	(wire
 		(pts
-			(xy 55.88 41.91) (xy 73.66 41.91)
-		)
-		(stroke
-			(width 0)
-			(type default)
-		)
-	)
-	(wire
-		(pts
 			(xy 77.47 74.93) (xy 115.57 74.93)
 		)
@@
 	(wire
 		(pts
-			(xy 133.35 63.5) (xy 133.35 82.55)
-		)
-		(stroke
-			(width 0)
-			(type default)
-		)
-	)
-	(wire
-		(pts
-			(xy 133.35 82.55) (xy 140.97 82.55)
+			(xy 137.16 55.88) (xy 154.94 55.88)
 		)
 		(stroke
@@
 	(wire
 		(pts
+			(xy 127 80.01) (xy 140.97 80.01)
+		)
+		(stroke
+			(width 0)
+			(type default)
+		)
+	)
+	(wire
+		(pts
 			(xy 97.79 63.5) (xy 97.79 67.31)
 		)
@@
 	(wire
 		(pts
+			(xy 154.94 48.26) (xy 154.94 55.88)
+		)
+		(stroke
+			(width 0)
+			(type default)
+		)
+	)
+	(wire
+		(pts
 			(xy 106.68 55.88) (xy 115.57 55.88)
 		)
@@
 	(wire
 		(pts
-			(xy 77.47 82.55) (xy 133.35 82.55)
+			(xy 77.47 82.55) (xy 137.16 82.55)
 		)
 		(stroke
@@
 	(wire
 		(pts
-			(xy 77.47 64.77) (xy 140.97 64.77)
+			(xy 77.47 64.77) (xy 88.9 64.77)
 		)
 		(stroke
@@
 		)
 	)
+	(bus
+		(pts
+			(xy 58.42 36.83) (xy 58.42 39.37)
+		)
+		(stroke
+			(width 0)
+			(type default)
+		)
+	)
 	(wire
 		(pts
@@
 	(wire
 		(pts
-			(xy 154.94 48.26) (xy 177.8 48.26)
-		)
-		(stroke
-			(width 0)
-			(type default)
-		)
-	)
-	(wire
-		(pts
 			(xy 208.28 87.63) (xy 204.47 87.63)
 		)
@@
 	(wire
 		(pts
-			(xy 133.35 55.88) (xy 154.94 55.88)
-		)
-		(stroke
-			(width 0)
-			(type default)
-		)
-	)
-	(wire
-		(pts
-			(xy 154.94 48.26) (xy 154.94 55.88)
+			(xy 127 55.88) (xy 137.16 55.88)
+		)
+		(stroke
+			(width 0)
+			(type default)
+		)
+	)
+	(wire
+		(pts
+			(xy 137.16 82.55) (xy 140.97 82.55)
+		)
+		(stroke
+			(width 0)
+			(type default)
+		)
+	)
+	(wire
+		(pts
+			(xy 154.94 48.26) (xy 158.75 48.26)
 		)
 		(stroke
@@
 		)
 	)
-	(label "DETECT"
-		(at 177.8 48.26 180)
-		(effects
-			(font
-				(size 1.27 1.27)
-			)
-			(justify right bottom)
-		)
-	)
 	(label "SDIO.DAT3"
 		(at 77.47 67.31 0)
@@
 			)
 			(justify right bottom)
-		)
-	)
-	(hierarchical_label "DETECT"
-		(shape input)
-		(at 55.88 41.91 180)
-		(effects
-			(font
-				(size 1.27 1.27)
-			)
-			(justify right)
 		)
 	)
@@
 		(dnp no)
 		(property "Reference" "R54"
-			(at 143.51 58.166 0)
-			(show_name no)
-			(do_not_autoplace no)
+			(at 139.954 58.42 0)
+			(show_name no)
+			(do_not_autoplace no)

Commit message: connecting i2c and uart bt/hdmi
Changed lines of the file:
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@@
 		)
 	)
-	(hierarchical_label "SDIO{DAT0 DAT1 DAT2 DAT3 CMD CLK}"
+	(hierarchical_label "SDIO{DAT0..3 CMD CLK}"
 		(shape input)
 		(at 57.15 22.86 180)
@@
 		)
 	)
-	(hierarchical_label "SDIO"
+	(hierarchical_label "SDIO{DAT0..3 CMD CLK}"
 		(shape input)
 		(at 53.34 60.96 180)
