File: HARDWARE/MINIHATv.0/HDMI.kicad_sch (KiCad schematic)
At the start: 28 parts, among them J4 HDMI_A, U11 TXB0104PW, U6 TFP410PAP

Commit message: mcu pwr/vcap ports, hdmi gpio, buses
Parts:
- R35: value 510 -> 510 1%
Connections:
- net LTDC_CEC: now also U11.11 (B3)
- net LTDC_HTPLG: now also U11.5 (A4); no longer J4.19 (HPD)
- net LTDC_HTPLG_5V: now reaches U11.10 (B4)
- net LTDC_HTPLG_5V: now also J4.19 (HPD)
- net MCU_LTDC_CEC: now reaches U11.4 (A3)
Other:
- moved on the sheet: U11
Changed lines of the file:
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@@
 	)
 	(junction
-		(at 255.27 118.11)
+		(at 226.06 110.49)
 		(diameter 0)
 		(color 0 0 0 0)
@@
 	(wire
 		(pts
-			(xy 267.97 133.35) (xy 271.78 133.35)
+			(xy 238.76 125.73) (xy 254 125.73)
 		)
 		(stroke
@@
 	(wire
 		(pts
+			(xy 254 130.81) (xy 238.76 130.81)
+		)
+		(stroke
+			(width 0)
+			(type default)
+		)
+	)
+	(wire
+		(pts
 			(xy 26.67 71.12) (xy 36.83 71.12)
 		)
@@
 	(wire
 		(pts
+			(xy 229.87 73.66) (xy 246.38 73.66)
+		)
+		(stroke
+			(width 0)
+			(type default)
+		)
+	)
+	(wire
+		(pts
 			(xy 109.22 134.62) (xy 111.76 134.62)
 		)
@@
 	(wire
 		(pts
+			(xy 254 135.89) (xy 238.76 135.89)
+		)
+		(stroke
+			(width 0)
+			(type default)
+		)
+	)
+	(wire
+		(pts
 			(xy 53.34 55.88) (xy 57.15 55.88)
 		)
@@
 		)
 	)
+	(wire
+		(pts
+			(xy 204.47 135.89) (xy 218.44 135.89)
+		)
+		(stroke
+			(width 0)
+			(type default)
+		)
+	)
 	(bus
 		(pts
@@
 	(wire
 		(pts
-			(xy 243.84 118.11) (xy 255.27 118.11)
+			(xy 214.63 110.49) (xy 226.06 110.49)
 		)
 		(stroke
@@
 	(wire
 		(pts
-			(xy 267.97 128.27) (xy 271.78 128.27)
+			(xy 238.76 120.65) (xy 254 120.65)
 		)
 		(stroke
@@
 	(wire
 		(pts
-			(xy 243.84 123.19) (xy 243.84 118.11)
+			(xy 214.63 115.57) (xy 214.63 110.49)
 		)
 		(stroke
@@
 	(wire
 		(pts
-			(xy 232.41 88.9) (xy 246.38 88.9)
+			(xy 229.87 88.9) (xy 246.38 88.9)
 		)
 		(stroke
@@
 	(wire
 		(pts
-			(xy 247.65 123.19) (xy 243.84 123.19)
+			(xy 218.44 115.57) (xy 214.63 115.57)
 		)
 		(stroke
@@
 		)
 	)
+	(label "LTDC_CEC"
+		(at 229.87 73.66 0)
+		(effects
+			(font
+				(size 1.27 1.27)
+			)
+			(justify left bottom)
+		)
+	)
 	(label "LTDC_R7"
 		(at 135.89 116.84 180)
@@
 		)
 	)
-	(label "LTDC_HTPLG"
-		(at 232.41 88.9 0)
+	(label "LTDC_HTPLG_5V"
+		(at 229.87 88.9 0)
 		(effects
 			(font
@@
 		)
 	)
+	(label "LTDC_HTPLG"
+		(at 204.47 135.89 0)
+		(effects
+			(font
+				(size 1.27 1.27)
+			)
+			(justify left bottom)
+		)
+	)
 	(label "TX2-"
 		(at 177.8 86.36 0)
@@
 		)
 	)
+	(label "LTDC_CEC"
+		(at 254 130.81 180)
+		(effects
+			(font
+				(size 1.27 1.27)
+			)
+			(justify right bottom)
+		)
+	)
+	(label "LTDC_HTPLG_5V"
+		(at 254 135.89 180)
+		(effects
+			(font
+				(size 1.27 1.27)
+			)
+			(justify right bottom)
+		)
+	)
 	(label "HDMI_SDA"
-		(at 271.78 133.35 0)
+		(at 254 125.73 180)
 		(effects
 			(font
 				(size 1.27 1.27)
 			)
-			(justify left bottom)
+			(justify right bottom)
 		)
 	)
@@
 	)
 	(label "HDMI_SCL"
-		(at 271.78 128.27 0)
+		(at 254 120.65 180)
 		(effects
 			(font
 				(size 1.27 1.27)
 			)
-			(justify left bottom)
+			(justify right bottom)
 		)
 	)
@@
 		)
 	)
-	(hierarchical_label "LTDC_CEC"
-		(shape output)
-		(at 246.38 73.66 180)
-		(effects
-			(font
-				(size 1.27 1.27)
-			)
-			(justify right)
-		)
-	)
 	(hierarchical_label "LTDC_MSEN"
 		(shape output)
@@
 		)
 	)
+	(hierarchical_label "MCU_LTDC_CEC"
+		(shape output)
+		(at 218.44 130.81 180)
+		(effects
+			(font
+				(size 1.27 1.27)
+			)
+			(justify right)
+		)
+	)
 	(hierarchical_label "{MCU_LTDC_BUS}"
 		(shape input)
@@
 	(hierarchical_label "HDMI_SCL"
 		(shape input)
-		(at 247.65 128.27 180)
+		(at 218.44 120.65 180)
 		(effects
 			(font
@@
 	(hierarchical_label "HDMI_SDA"
 		(shape input)
-		(at 247.65 133.35 180)
+		(at 218.44 125.73 180)
 		(effects
 			(font
@@
 	(symbol
 		(lib_id "Logic_LevelTranslator:TXB0104PW")
-		(at 257.81 135.89 0)
+		(at 228.6 128.27 0)
 		(unit 1)
 		(body_style 1)
@@
 		(fields_autoplaced yes)
 		(property "Reference" "U11"
-			(at 259.9533 153.67 0)
+			(at 230.7433 146.05 0)
 			(show_name no)
 			(do_not_autoplace no)
@@
 		)
 		(property "Value" "TXB0104PW"
-			(at 259.9533 156.21 0)
+			(at 230.7433 148.59 0)
 			(show_name no)
 			(do_not_autoplace no)
@@
 		)
 		(property "Footprint" "Package_SO:TSSOP-14_4.4x5mm_P0.65mm"
-			(at 257.81 154.94 0)
+			(at 228.6 147.32 0)
 			(hide yes)
 			(show_name no)
@@
 		)
 		(property "Datasheet" "http://www.ti.com/lit/ds/symlink/txb0104.pdf"
-			(at 260.604 133.477 0)
+			(at 231.394 125.857 0)
 			(hide yes)
 			(show_name no)
@@
 		)
 		(property "Description" "4-Bit Bidirectional Voltage-Level Translator, Auto Direction Sensing and ±15-kV ESD Protection, 1.2 - 3.6V APort, 1.65 - 5.5V BPort, TSSOP-14"
-			(at 257.81 135.89 0)
+			(at 228.6 128.27 0)
 			(hide yes)
 			(show_name no)
@@
 			)
 		)
-		(property "Value" "510"
+		(property "Value" "510 1%"
 			(at 177.8 53.848 90)
 			(show_name no)
@@
 	(symbol
 		(lib_id "power:+3V3")
-		(at 260.35 118.11 0)
+		(at 231.14 110.49 0)
 		(unit 1)
 		(body_style 1)
@@
 		(dnp no)
 		(property "Reference" "#PWR0107"
-			(at 260.35 121.92 0)
+			(at 231.14 114.3 0)
 			(hide yes)
 			(show_name no)
@@
 		)
 		(property "Value" "+5V"
-			(at 258.826 112.776 0)
+			(at 229.616 105.156 0)
 			(show_name no)
 			(do_not_autoplace no)
@@
 		)
 		(property "Footprint" ""
-			(at 260.35 118.11 0)
+			(at 231.14 110.49 0)
 			(hide yes)
 			(show_name no)
@@
 		)
 		(property "Datasheet" ""
-			(at 260.35 118.11 0)
+			(at 231.14 110.49 0)
 			(hide yes)
 			(show_name no)
@@
 		)
 		(property "Description" "Power symbol creates a global label with name \"+3V3\""
-			(at 260.35 118.11 0)
+			(at 231.14 110.49 0)
 			(hide yes)
 			(show_name no)
@@
 	(symbol
 		(lib_id "power:+3V3")
-		(at 255.27 118.11 0)
+		(at 226.06 110.49 0)
 		(unit 1)
 		(body_style 1)
@@
 		(fields_autoplaced yes)
 		(property "Reference" "#PWR09"
-			(at 255.27 121.92 0)
+			(at 226.06 114.3 0)
 			(hide yes)
 			(show_name no)
@@
 		)
 		(property "Value" "+3V3"
-			(at 255.27 113.03 0)
+			(at 226.06 105.41 0)
 			(show_name no)
 			(do_not_autoplace no)
@@
 		)
 		(property "Footprint" ""
-			(at 255.27 118.11 0)
+			(at 226.06 110.49 0)
 			(hide yes)
 			(show_name no)
@@
 		)
 		(property "Datasheet" ""
-			(at 255.27 118.11 0)
+			(at 226.06 110.49 0)
 			(hide yes)
 			(show_name no)
@@
 		)
 		(property "Description" "Power symbol creates a global label with name \"+3V3\""
-			(at 255.27 118.11 0)
+			(at 226.06 110.49 0)
 			(hide yes)
 			(show_name no)
@@
 	(symbol
 		(lib_id "power:GND")
-		(at 257.81 153.67 0)
+		(at 228.6 146.05 0)
 		(unit 1)
 		(body_style 1)
@@
 		(fields_autoplaced yes)
 		(property "Reference" "#PWR0110"
-			(at 257.81 160.02 0)
+			(at 228.6 152.4 0)
 			(hide yes)
 			(show_name no)
@@
 		)
 		(property "Value" "GND"
-			(at 257.81 158.75 0)
+			(at 228.6 151.13 0)
 			(show_name no)
 			(do_not_autoplace no)
@@
 		)
 		(property "Footprint" ""
-			(at 257.81 153.67 0)
+			(at 228.6 146.05 0)
 			(hide yes)
 			(show_name no)
@@
 		)
 		(property "Datasheet" ""
-			(at 257.81 153.67 0)
+			(at 228.6 146.05 0)
 			(hide yes)
 			(show_name no)
@@
 		)
 		(property "Description" "Power symbol creates a global label with name \"GND\" , ground"
-			(at 257.81 153.67 0)
+			(at 228.6 146.05 0)
 			(hide yes)
 			(show_name no)

Commit message: BT 1V2 lowdrop added, fdcan pinned to mcu, usb status led added
Parts:
- added C101: 100n, symbol Device:C_Small
Connections:
- net GND: now also C101.2
- net at R36.2, R37.1, U6.3 (VREF): now also C101.1
Changed lines of the file:
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@@
 	(wire
 		(pts
-			(xy 238.76 125.73) (xy 254 125.73)
+			(xy 238.76 125.73) (xy 255.27 125.73)
 		)
 		(stroke
@@
 	(wire
 		(pts
+			(xy 213.36 125.73) (xy 218.44 125.73)
+		)
+		(stroke
+			(width 0)
+			(type default)
+		)
+	)
+	(wire
+		(pts
 			(xy 171.45 88.9) (xy 187.96 88.9)
 		)
@@
 	(wire
 		(pts
-			(xy 254 130.81) (xy 238.76 130.81)
+			(xy 255.27 130.81) (xy 238.76 130.81)
 		)
 		(stroke
@@
 	(wire
 		(pts
-			(xy 254 135.89) (xy 238.76 135.89)
+			(xy 255.27 135.89) (xy 238.76 135.89)
 		)
 		(stroke
@@
 	(wire
 		(pts
-			(xy 204.47 135.89) (xy 218.44 135.89)
+			(xy 203.2 135.89) (xy 218.44 135.89)
 		)
 		(stroke
@@
 	(wire
 		(pts
+			(xy 213.36 120.65) (xy 218.44 120.65)
+		)
+		(stroke
+			(width 0)
+			(type default)
+		)
+	)
+	(wire
+		(pts
 			(xy 53.34 71.12) (xy 53.34 72.39)
 		)
@@
 	(wire
 		(pts
+			(xy 201.93 52.07) (xy 201.93 50.8)
+		)
+		(stroke
+			(width 0)
+			(type default)
+		)
+	)
+	(wire
+		(pts
 			(xy 52.07 25.4) (xy 72.39 25.4)
 		)
@@
 	(wire
 		(pts
-			(xy 238.76 120.65) (xy 254 120.65)
+			(xy 238.76 120.65) (xy 255.27 120.65)
 		)
 		(stroke
@@
 		(pts
 			(xy 123.19 86.36) (xy 135.89 86.36)
+		)
+		(stroke
+			(width 0)
+			(type default)
+		)
+	)
+	(wire
+		(pts
+			(xy 201.93 50.8) (xy 191.77 50.8)
 		)
 		(stroke
@@
 	)
 	(label "LTDC_HTPLG"
-		(at 204.47 135.89 0)
+		(at 203.2 135.89 0)
 		(effects
 			(font
@@
 	)
 	(label "LTDC_CEC"
-		(at 254 130.81 180)
+		(at 255.27 130.81 180)
 		(effects
 			(font
@@
 	)
 	(label "LTDC_HTPLG_5V"
-		(at 254 135.89 180)
+		(at 255.27 135.89 180)
 		(effects
 			(font
@@
 	)
 	(label "HDMI_SDA"
-		(at 254 125.73 180)
+		(at 255.27 125.73 180)
 		(effects
 			(font
@@
 	)
 	(label "HDMI_SCL"
-		(at 254 120.65 180)
+		(at 255.27 120.65 180)
 		(effects
 			(font
@@
 	(hierarchical_label "HDMI_SCL"
 		(shape input)
-		(at 218.44 120.65 180)
+		(at 213.36 120.65 180)
 		(effects
 			(font
@@
 	(hierarchical_label "HDMI_SDA"
 		(shape input)
-		(at 218.44 125.73 180)
+		(at 213.36 125.73 180)
 		(effects
 			(font
@@
 	)
 	(symbol
+		(lib_id "Device:C_Small")
+		(at 201.93 54.61 0)
+		(unit 1)
+		(body_style 1)
+		(exclude_from_sim no)
+		(in_bom yes)
+		(on_board yes)
+		(in_pos_files yes)
+		(dnp no)
+		(fields_autoplaced yes)
+		(property "Reference" "C101"
+			(at 204.47 53.3462 0)
+			(show_name no)
+			(do_not_autoplace no)
+			(effects
+				(font
+					(size 1.27 1.27)
+				)
+				(justify left)
+			)
+		)
+		(property "Value" "100n"
+			(at 204.47 55.8862 0)
+			(show_name no)
+			(do_not_autoplace no)
+			(effects
+				(font
+					(size 1.27 1.27)
+				)
+				(justify left)
+			)
+		)
+		(property "Footprint" ""
+			(at 201.93 54.61 0)
+			(hide yes)
+			(show_name no)
+			(do_not_autoplace no)
+			(effects
+				(font
+					(size 1.27 1.27)
+				)
+			)
+		)
+		(property "Datasheet" ""
+			(at 201.93 54.61 0)
+			(hide yes)
+			(show_name no)
+			(do_not_autoplace no)
+			(effects
+				(font
+					(size 1.27 1.27)
+				)
+			)
+		)
+		(property "Description" "Unpolarized capacitor, small symbol"
+			(at 201.93 54.61 0)
+			(hide yes)
+			(show_name no)
+			(do_not_autoplace no)
+			(effects
+				(font
+					(size 1.27 1.27)
+				)
+			)
+		)
+		(pin "1"
+		)
+		(pin "2"
+		)
+		(instances
+			(project "MINIHATv.0"
+				(path "/19041ef4-1d16-4363-8780-721ad9f20b33/92951603-bc2e-4dd1-8377-ba7c43df3b1e"
+					(reference "C101")
+					(unit 1)
+				)
+			)
+		)
+	)
+	(symbol
 		(lib_id "power:+3V3")
 		(at 191.77 44.45 0)
@@
 					(unit 1)
 				)
+			)
+		)
+	)
+	(symbol
+		(lib_id "power:GND")
+		(at 201.93 57.15 0)
+		(unit 1)
+		(body_style 1)
+		(exclude_from_sim no)
+		(in_bom yes)
+		(on_board yes)
+		(in_pos_files yes)
+		(dnp no)
+		(fields_autoplaced yes)
+		(property "Reference" "#PWR0142"
+			(at 201.93 63.5 0)
+			(hide yes)
+			(show_name no)
+			(do_not_autoplace no)
+			(effects
+				(font
+					(size 1.27 1.27)
+				)
+			)
+		)
+		(property "Value" "GND"
+			(at 201.93 62.23 0)
+			(show_name no)
+			(do_not_autoplace no)
+			(effects
+				(font
+					(size 1.27 1.27)
+				)
+			)
+		)
+		(property "Footprint" ""
+			(at 201.93 57.15 0)
+			(hide yes)
+			(show_name no)
+			(do_not_autoplace no)
+			(effects
+				(font
+					(size 1.27 1.27)
+				)
+			)
+		)
+		(property "Datasheet" ""
+			(at 201.93 57.15 0)
+			(hide yes)
+			(show_name no)
+			(do_not_autoplace no)
+			(effects
+				(font
+					(size 1.27 1.27)
+				)
+			)
+		)
+		(property "Description" "Power symbol creates a global label with name \"GND\" , ground"
+			(at 201.93 57.15 0)
+			(hide yes)
+			(show_name no)
+			(do_not_autoplace no)
+			(effects
+				(font
+					(size 1.27 1.27)
+				)
+			)
+		)
+		(pin "1"
+		)
+		(instances
+			(project "MINIHATv.0"
+				(path "/19041ef4-1d16-4363-8780-721ad9f20b33/92951603-bc2e-4dd1-8377-ba7c43df3b1e"
+					(reference "#PWR0142")
+					(unit 1)
+				)
