File: HARDWARE/MINIHATv.0/usb.kicad_sch (KiCad schematic)
At the start: 8 parts, among them P1 USB_C_Plug, U4 USBLC6-2P6

Commit message: added normal buses
Other:
- moved on the sheet: C12, C13, P1, R40, R41, R42, R43, U4

Commit message: added sdram and usb pages to top page
Parts:
- renumbered C12 to C59, C13 to C60, P1 to P2, R42 to R4, R43 to R5, R40 to R82, R41 to R83, U4 to U10
Changed lines of the file:
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@@
 		(instances
 			(project "MINIHATv.0"
-				(path "/19041ef4-1d16-4363-8780-721ad9f20b33/7587cd4c-2835-4070-8105-8c12f1b1d372"
+				(path "/19041ef4-1d16-4363-8780-721ad9f20b33/777e9115-49d2-40e9-92df-ea6663fef183"
 					(reference "#PWR039")
 					(unit 1)
@@
 		(instances
 			(project "MINIHATv.0"
-				(path "/19041ef4-1d16-4363-8780-721ad9f20b33/7587cd4c-2835-4070-8105-8c12f1b1d372"
+				(path "/19041ef4-1d16-4363-8780-721ad9f20b33/777e9115-49d2-40e9-92df-ea6663fef183"
 					(reference "#PWR033")
 					(unit 1)
@@
 		(dnp no)
 		(fields_autoplaced yes)
-		(property "Reference" "P1"
+		(property "Reference" "P2"
 			(at 149.86 81.2799 0)
 			(show_name no)
@@
 		(instances
 			(project "MINIHATv.0"
-				(path "/19041ef4-1d16-4363-8780-721ad9f20b33/7587cd4c-2835-4070-8105-8c12f1b1d372"
-					(reference "P1")
+				(path "/19041ef4-1d16-4363-8780-721ad9f20b33/777e9115-49d2-40e9-92df-ea6663fef183"
+					(reference "P2")
 					(unit 1)
 				)
@@
 		(dnp no)
 		(fields_autoplaced yes)
-		(property "Reference" "C13"
+		(property "Reference" "C60"
 			(at 104.14 44.4499 0)
 			(show_name no)
@@
 		(instances
 			(project "MINIHATv.0"
-				(path "/19041ef4-1d16-4363-8780-721ad9f20b33/7587cd4c-2835-4070-8105-8c12f1b1d372"
-					(reference "C13")
+				(path "/19041ef4-1d16-4363-8780-721ad9f20b33/777e9115-49d2-40e9-92df-ea6663fef183"
+					(reference "C60")
 					(unit 1)
 				)
@@
 		(instances
 			(project "MINIHATv.0"
-				(path "/19041ef4-1d16-4363-8780-721ad9f20b33/7587cd4c-2835-4070-8105-8c12f1b1d372"
+				(path "/19041ef4-1d16-4363-8780-721ad9f20b33/777e9115-49d2-40e9-92df-ea6663fef183"
 					(reference "#PWR034")
 					(unit 1)
@@
 		(dnp no)
 		(fields_autoplaced yes)
-		(property "Reference" "R43"
+		(property "Reference" "R5"
 			(at 86.36 48.2599 0)
 			(show_name no)
@@
 		(instances
 			(project "MINIHATv.0"
-				(path "/19041ef4-1d16-4363-8780-721ad9f20b33/7587cd4c-2835-4070-8105-8c12f1b1d372"
-					(reference "R43")
+				(path "/19041ef4-1d16-4363-8780-721ad9f20b33/777e9115-49d2-40e9-92df-ea6663fef183"
+					(reference "R5")
 					(unit 1)
 				)
@@
 		(instances
 			(project "MINIHATv.0"
-				(path "/19041ef4-1d16-4363-8780-721ad9f20b33/7587cd4c-2835-4070-8105-8c12f1b1d372"
+				(path "/19041ef4-1d16-4363-8780-721ad9f20b33/777e9115-49d2-40e9-92df-ea6663fef183"
 					(reference "#PWR038")
 					(unit 1)
@@
 		(in_pos_files yes)
 		(dnp no)
-		(property "Reference" "U4"
+		(property "Reference" "U10"
 			(at 82.55 76.708 0)
 			(show_name no)
@@
 		(instances
 			(project "MINIHATv.0"
-				(path "/19041ef4-1d16-4363-8780-721ad9f20b33/7587cd4c-2835-4070-8105-8c12f1b1d372"
-					(reference "U4")
+				(path "/19041ef4-1d16-4363-8780-721ad9f20b33/777e9115-49d2-40e9-92df-ea6663fef183"
+					(reference "U10")
 					(unit 1)
 				)
@@
 		(instances
 			(project "MINIHATv.0"
-				(path "/19041ef4-1d16-4363-8780-721ad9f20b33/7587cd4c-2835-4070-8105-8c12f1b1d372"
+				(path "/19041ef4-1d16-4363-8780-721ad9f20b33/777e9115-49d2-40e9-92df-ea6663fef183"
 					(reference "#PWR032")
 					(unit 1)
@@
 		(instances
 			(project "MINIHATv.0"
-				(path "/19041ef4-1d16-4363-8780-721ad9f20b33/7587cd4c-2835-4070-8105-8c12f1b1d372"
+				(path "/19041ef4-1d16-4363-8780-721ad9f20b33/777e9115-49d2-40e9-92df-ea6663fef183"
 					(reference "#PWR041")
 					(unit 1)
@@
 		(instances
 			(project "MINIHATv.0"
-				(path "/19041ef4-1d16-4363-8780-721ad9f20b33/7587cd4c-2835-4070-8105-8c12f1b1d372"
+				(path "/19041ef4-1d16-4363-8780-721ad9f20b33/777e9115-49d2-40e9-92df-ea6663fef183"
 					(reference "#PWR037")
 					(unit 1)
@@
 		(instances
 			(project "MINIHATv.0"
-				(path "/19041ef4-1d16-4363-8780-721ad9f20b33/7587cd4c-2835-4070-8105-8c12f1b1d372"
+				(path "/19041ef4-1d16-4363-8780-721ad9f20b33/777e9115-49d2-40e9-92df-ea6663fef183"
 					(reference "#PWR040")
 					(unit 1)
@@
 		(instances
 			(project "MINIHATv.0"
-				(path "/19041ef4-1d16-4363-8780-721ad9f20b33/7587cd4c-2835-4070-8105-8c12f1b1d372"
+				(path "/19041ef4-1d16-4363-8780-721ad9f20b33/777e9115-49d2-40e9-92df-ea6663fef183"
 					(reference "#PWR036")
 					(unit 1)
@@
 		(in_pos_files yes)
 		(dnp no)
-		(property "Reference" "R41"
+		(property "Reference" "R83"
 			(at 110.744 59.944 90)
 			(show_name no)
@@
 		(instances
 			(project "MINIHATv.0"
-				(path "/19041ef4-1d16-4363-8780-721ad9f20b33/7587cd4c-2835-4070-8105-8c12f1b1d372"
-					(reference "R41")
+				(path "/19041ef4-1d16-4363-8780-721ad9f20b33/777e9115-49d2-40e9-92df-ea6663fef183"
+					(reference "R83")
 					(unit 1)
 				)
@@
 		(instances
 			(project "MINIHATv.0"
-				(path "/19041ef4-1d16-4363-8780-721ad9f20b33/7587cd4c-2835-4070-8105-8c12f1b1d372"
+				(path "/19041ef4-1d16-4363-8780-721ad9f20b33/777e9115-49d2-40e9-92df-ea6663fef183"
 					(reference "#PWR035")
 					(unit 1)
@@
 		(dnp no)
 		(fields_autoplaced yes)
-		(property "Reference" "R42"
+		(property "Reference" "R4"
 			(at 86.36 35.5599 0)
 			(show_name no)
@@
 		(instances
 			(project "MINIHATv.0"
-				(path "/19041ef4-1d16-4363-8780-721ad9f20b33/7587cd4c-2835-4070-8105-8c12f1b1d372"
-					(reference "R42")
+				(path "/19041ef4-1d16-4363-8780-721ad9f20b33/777e9115-49d2-40e9-92df-ea6663fef183"
+					(reference "R4")
 					(unit 1)
 				)
@@
 		(dnp no)
 		(fields_autoplaced yes)
-		(property "Reference" "C12"
+		(property "Reference" "C59"
 			(at 76.2 48.2599 0)
 			(show_name no)
@@
 		(instances
 			(project "MINIHATv.0"
-				(path "/19041ef4-1d16-4363-8780-721ad9f20b33/7587cd4c-2835-4070-8105-8c12f1b1d372"
-					(reference "C12")
+				(path "/19041ef4-1d16-4363-8780-721ad9f20b33/777e9115-49d2-40e9-92df-ea6663fef183"
+					(reference "C59")
 					(unit 1)
 				)
@@
 		(in_pos_files yes)
 		(dnp no)
-		(property "Reference" "R40"
+		(property "Reference" "R82"
 			(at 110.744 57.404 90)
 			(show_name no)
@@
 		(instances
 			(project "MINIHATv.0"
-				(path "/19041ef4-1d16-4363-8780-721ad9f20b33/7587cd4c-2835-4070-8105-8c12f1b1d372"
-					(reference "R40")
-					(unit 1)
-				)
+				(path "/19041ef4-1d16-4363-8780-721ad9f20b33/777e9115-49d2-40e9-92df-ea6663fef183"
+					(reference "R82")
+					(unit 1)
+				)

Commit message: BT 1V2 lowdrop added, fdcan pinned to mcu, usb status led added
Parts:
- added D11: LED R, symbol Device:LED
- added R94: 220, symbol Device:R_Small
Connections:
- net GND: now also R94.2
- net USB_SENSE: now also D11.2 (A)
- new net: D11.1 (K), R94.1
